Commit message: adding some jank inertias

File: assets/foosball_table/foosball_table.urdf (robot description, URDF)
Before this commit: robot foosball_table, 17 links, 16 joints
Links:
- link 2_bar_team_1: mass None -> 0.7638
- link 2_bar_team_2: mass None -> 0.7638
- link 3_bar_team_1: mass None -> 0.7638
- link 3_bar_team_2: mass None -> 0.7638
- link 5_bar_team_1: mass None -> 0.7638
- link 5_bar_team_2: mass None -> 0.7638
- link goalie_team_1: mass None -> 0.7638
- link goalie_team_2: mass None -> 0.7638

Commit message: splitting meshes into teams, adding script to change team colors

File: assets/foosball_table/foosball_table.urdf (robot description, URDF)
Before this commit: robot foosball_table, 17 links, 16 joints
Links:
- link 2_bar_team_1: geometry collision mesh filename=meshes/2-bar-centered_team_1.obj scale=1 1 1; visual mesh filename=meshes/2-bar-centered_team_1.obj scale=1 1 1
- link 2_bar_team_2: geometry collision mesh filename=meshes/2-bar-centered_team_2.obj scale=1 1 1; visual mesh filename=meshes/2-bar-centered_team_2.obj scale=1 1 1
- link 3_bar_team_1: geometry collision mesh filename=meshes/3-bar-centered_team_1.obj scale=1 1 1; visual mesh filename=meshes/3-bar-centered_team_1.obj scale=1 1 1
- link 3_bar_team_2: geometry collision mesh filename=meshes/3-bar-centered_team_2.obj scale=1 1 1; visual mesh filename=meshes/3-bar-centered_team_2.obj scale=1 1 1
- link 5_bar_team_1: geometry collision mesh filename=meshes/5-bar-centered_team_1.obj scale=1 1 1; visual mesh filename=meshes/5-bar-centered_team_1.obj scale=1 1 1
- link 5_bar_team_2: geometry collision mesh filename=meshes/5-bar-centered_team_2.obj scale=1 1 1; visual mesh filename=meshes/5-bar-centered_team_2.obj scale=1 1 1
- link goalie_team_1: geometry collision mesh filename=meshes/1-bar-centered.obj_team_1 scale=1 1 1; visual mesh filename=meshes/1-bar-centered_team_1.obj scale=1 1 1
- link goalie_team_2: geometry collision mesh filename=meshes/1-bar-centered_team_2.obj scale=1 1 1; visual mesh filename=meshes/1-bar-centered_team_2.obj scale=1 1 1
